Commit message: Edited the Notebooks 3, 6 in the section 1

File: section_1_introduction_and_tools/Robot.urdf (robot description, URDF)
Before this commit: robot robot, 6 links, 5 joints
Links:
- removed link caster_wheel
- added link sphere_wheel; collision sphere radius=0.05; visual sphere radius=0.05
Joints:
- removed joint caster_wheel_joint
- added joint sphere_wheel_joint: type fixed, parent chassis, child sphere_wheel, origin xyz=0.24 0 0 rpy=0 0 0
